Commit message: Deleted some things to save space which are not needed for our purposes such as the urdf files and meshes of the turrets made by interbotix

File: src/interbotix_ros_turrets/interbotix_ros_xsturrets/interbotix_xsturret_descriptions/urdf/Full_Turret_Cam.urdf.xacro (robot description, xacro)
@@ -186,5 +186,5 @@
   </transmission>
   <joint name="camera" type="fixed">
-    <origin rpy="${-pi/2} 0 ${-pi/2}" xyz="0.0312 0 0.03"/>
+    <origin rpy="${-pi/2} ${-pi/2} ${-pi/2}" xyz="0.00035552 0.000776777777232895 0.004546"/>
     <parent link="shooter_link"/>
     <child link="camera_link"/>
@@ -192,14 +192,14 @@
   <link name="camera_link">
     <visual>
+      <origin rpy="0 0 0" xyz="0 0.0006777777232895 0.00152595494140505"/>
+      <geometry>
+        <mesh filename="package://interbotix_xsturret_descriptions/meshes/pxxls_cam_meshes/pxxls_cam_camera.stl" scale="0.001 0.001 0.001"/>
+      </geometry>
+    </visual>
+    <collision>
       <origin rpy="0 0 0" xyz="0 0 0"/>
       <geometry>
         <mesh filename="package://interbotix_xsturret_descriptions/meshes/pxxls_cam_meshes/pxxls_cam_camera.stl" scale="0.001 0.001 0.001"/>
       </geometry>
-    </visual>
-    <collision>
-      <origin rpy="0 0 0" xyz="0 0 0"/>
-      <geometry>
-        <mesh filename="package://interbotix_xsturret_descriptions/meshes/pxxls_cam_meshes/pxxls_cam_camera.stl" scale="0.001 0.001 0.001"/>
-      </geometry>
     </collision>
   </link>
